File: hardware/YouHaveThePowerKiCadProject/YouHaveThePowerKiCadProject.kicad_sch (KiCad schematic)
At the start: 0 parts

Commit message: added inital docs and fw folder
Parts:
- added U1: STM32H755ZITx, Package_QFP:LQFP-144_20x20mm_P0.5mm, symbol MCU_ST_STM32H7:STM32H755ZITx
Connections:
- new net: U1.104 (VSS), U1.118 (VSS), U1.12 (VSS), U1.128 (VSS), U1.141 (VSS), U1.18 (VSS), U1.33 (VSS), U1.41 (VSS), U1.55 (VSS), U1.6 (VSS), U1.69 (VSS), U1.80 (VSS)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
